File: zxmidi.kicad_sch (KiCad schematic)
At the start: 6 parts, among them J1 RJ45, J2 DIN-5_180degree, Q1 BC337

Commit message: Error fix
Parts:
- removed J1: RJ45, Connector_RJ:RJ45_Amphenol_54602-x08_Horizontal, symbol Connector:RJ45
- added J1: RJ45, ZXMidi:RJ45_Amphenol_54602-x08_Horizontal, symbol zx_midi:RJ45
- J2: symbol Connector:DIN-5_180degree -> zx_midi:DIN-5_180degree
- Q1: footprint Package_TO_SOT_THT:TO-92_Inline -> ZXMidi:TO-92_Inline; symbol Transistor_BJT:BC337 -> zx_midi:BC337
- R1: renamed from R3; footprint Resistor_THT:R_Axial_DIN0207_L6.3mm_D2.5mm_P10.16mm_Horizontal -> ZXMidi:R_Axial_DIN0207_L6.3mm_D2.5mm_P10.16mm_Horizontal; symbol Device:R -> zx_midi:R
- R2: renamed from R1; footprint Resistor_THT:R_Axial_DIN0207_L6.3mm_D2.5mm_P10.16mm_Horizontal -> ZXMidi:R_Axial_DIN0207_L6.3mm_D2.5mm_P10.16mm_Horizontal; symbol Device:R -> zx_midi:R
- R3: renamed from R2; footprint Resistor_THT:R_Axial_DIN0207_L6.3mm_D2.5mm_P10.16mm_Horizontal -> ZXMidi:R_Axial_DIN0207_L6.3mm_D2.5mm_P10.16mm_Horizontal; symbol Device:R -> zx_midi:R
Connections:
- net at R2.1: now also J1.4
- net at Q1.3 (E): now also J1.8
- net at R1.1: now also J1.3
- no-connect marks 8 -> 14
Changed lines of the file:
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@@
 (kicad_sch (version 20230121) (generator eeschema)
   (paper "A4")
+  (no_connect (at 31.115 27.305))
+  (no_connect (at 41.275 27.305))
+  (no_connect (at 33.655 27.305))
+  (no_connect (at 28.575 27.305))
+  (no_connect (at 38.735 27.305))
   (no_connect (at 45.085 32.385))
   (no_connect (at 99.06 33.655))
@@
   (no_connect (at 99.06 48.895))
   (no_connect (at 45.085 42.545))
+  (no_connect (at 36.195 27.305))
   (no_connect (at 45.085 45.085))
   (no_connect (at 45.085 47.625))
@@
     (stroke (width 0) (type default))
   )
-  (symbol (lib_id "Device:R") (at 55.245 40.005 90) (unit 1)
+  (symbol (lib_id "zx_midi:RJ45") (at 34.925 40.005 0) (mirror x) (unit 1)
+    (in_bom yes) (on_board yes) (dnp no)
+    (property "Reference" "J1" (at 34.925 57.15 0)
+      (effects (font (size 1.27 1.27)))
+    )
+    (property "Value" "RJ45" (at 34.925 54.61 0)
+      (effects (font (size 1.27 1.27)))
+    )
+    (property "Footprint" "ZXMidi:RJ45_Amphenol_54602-x08_Horizontal" (at 34.925 40.64 90)
+      (effects (font (size 1.27 1.27)) hide)
+    )
+    (property "Datasheet" "~" (at 34.925 40.64 90)
+      (effects (font (size 1.27 1.27)) hide)
+    )
+    (pin "1")
+    (pin "2")
+    (pin "3")
+    (pin "4")
+    (pin "5")
+    (pin "6")
+    (pin "7")
+    (pin "8")
+    (pin "11")
+    (pin "14")
+    (pin "12")
+    (pin "13")
+    (pin "9")
+    (pin "10")
+    (instances
+      (project "zxmidi"
+        (path "/0ef5500a-5958-4cb0-a7eb-d57b0bfb179a"
+          (reference "J1") (unit 1)
+        )
+      )
+    )
+  )
+  (symbol (lib_id "zx_midi:R") (at 55.245 40.005 90) (unit 1)
     (in_bom yes) (on_board yes) (dnp no) (fields_autoplaced)
-    (property "Reference" "R1" (at 55.245 34.925 90)
+    (property "Reference" "R2" (at 55.245 34.925 90)
       (effects (font (size 1.27 1.27)))
     )
@@
       (effects (font (size 1.27 1.27)))
     )
-    (property "Footprint" "Resistor_THT:R_Axial_DIN0207_L6.3mm_D2.5mm_P10.16mm_Horizontal" (at 55.245 41.783 90)
+    (property "Footprint" "ZXMidi:R_Axial_DIN0207_L6.3mm_D2.5mm_P10.16mm_Horizontal" (at 55.245 41.783 90)
       (effects (font (size 1.27 1.27)) hide)
     )
     (property "Datasheet" "~" (at 55.245 40.005 0)
-      (effects (font (size 1.27 1.27)) hide)
-    )
-    (pin "1")
-    (pin "2")
-    (instances
-      (project "zxmidi"
-        (path "/0ef5500a-5958-4cb0-a7eb-d57b0bfb179a"
-          (reference "R1") (unit 1)
-        )
-      )
-    )
-  )
-  (symbol (lib_id "Device:R") (at 83.185 27.305 90) (unit 1)
-    (in_bom yes) (on_board yes) (dnp no) (fields_autoplaced)
-    (property "Reference" "R2" (at 83.185 22.225 90)
-      (effects (font (size 1.27 1.27)))
-    )
-    (property "Value" "220" (at 83.185 24.765 90)
-      (effects (font (size 1.27 1.27)))
-    )
-    (property "Footprint" "Resistor_THT:R_Axial_DIN0207_L6.3mm_D2.5mm_P10.16mm_Horizontal" (at 83.185 29.083 90)
-      (effects (font (size 1.27 1.27)) hide)
-    )
-    (property "Datasheet" "~" (at 83.185 27.305 0)
       (effects (font (size 1.27 1.27)) hide)
     )
@@
     )
   )
-  (symbol (lib_id "Connector:RJ45") (at 34.925 42.545 0) (unit 1)
+  (symbol (lib_id "zx_midi:R") (at 83.185 27.305 90) (unit 1)
     (in_bom yes) (on_board yes) (dnp no) (fields_autoplaced)
-    (property "Reference" "J1" (at 34.925 25.4 0)
+    (property "Reference" "R3" (at 83.185 22.225 90)
       (effects (font (size 1.27 1.27)))
     )
-    (property "Value" "RJ45" (at 34.925 27.94 0)
+    (property "Value" "220" (at 83.185 24.765 90)
       (effects (font (size 1.27 1.27)))
     )
-    (property "Footprint" "Connector_RJ:RJ45_Amphenol_54602-x08_Horizontal" (at 34.925 41.91 90)
+    (property "Footprint" "ZXMidi:R_Axial_DIN0207_L6.3mm_D2.5mm_P10.16mm_Horizontal" (at 83.185 29.083 90)
       (effects (font (size 1.27 1.27)) hide)
     )
-    (property "Datasheet" "~" (at 34.925 41.91 90)
+    (property "Datasheet" "~" (at 83.185 27.305 0)
       (effects (font (size 1.27 1.27)) hide)
     )
     (pin "1")
     (pin "2")
-    (pin "3")
-    (pin "4")
-    (pin "5")
-    (pin "6")
-    (pin "7")
-    (pin "8")
     (instances
       (project "zxmidi"
         (path "/0ef5500a-5958-4cb0-a7eb-d57b0bfb179a"
-          (reference "J1") (unit 1)
+          (reference "R3") (unit 1)
         )
       )
     )
   )
-  (symbol (lib_id "Transistor_BJT:BC337") (at 67.945 40.005 0) (unit 1)
+  (symbol (lib_id "zx_midi:BC337") (at 67.945 40.005 0) (unit 1)
     (in_bom yes) (on_board yes) (dnp no) (fields_autoplaced)
     (property "Reference" "Q1" (at 73.66 39.37 0)
@@
       (effects (font (size 1.27 1.27)) (justify left))
     )
-    (property "Footprint" "Package_TO_SOT_THT:TO-92_Inline" (at 73.025 41.91 0)
+    (property "Footprint" "ZXMidi:TO-92_Inline" (at 73.025 41.91 0)
       (effects (font (size 1.27 1.27) italic) (justify left) hide)
     )
@@
     )
   )
-  (symbol (lib_id "Device:R") (at 83.185 56.515 90) (unit 1)
+  (symbol (lib_id "zx_midi:R") (at 83.185 56.515 90) (unit 1)
     (in_bom yes) (on_board yes) (dnp no) (fields_autoplaced)
-    (property "Reference" "R3" (at 83.185 51.435 90)
+    (property "Reference" "R1" (at 83.185 51.435 90)
       (effects (font (size 1.27 1.27)))
     )
@@
       (effects (font (size 1.27 1.27)))
     )
-    (property "Footprint" "Resistor_THT:R_Axial_DIN0207_L6.3mm_D2.5mm_P10.16mm_Horizontal" (at 83.185 58.293 90)
+    (property "Footprint" "ZXMidi:R_Axial_DIN0207_L6.3mm_D2.5mm_P10.16mm_Horizontal" (at 83.185 58.293 90)
       (effects (font (size 1.27 1.27)) hide)
     )
@@
       (project "zxmidi"
         (path "/0ef5500a-5958-4cb0-a7eb-d57b0bfb179a"
-          (reference "R3") (unit 1)
+          (reference "R1") (unit 1)
         )
       )
     )
   )
-  (symbol (lib_id "Connector:DIN-5_180degree") (at 99.06 41.275 90) (unit 1)
+  (symbol (lib_id "zx_midi:DIN-5_180degree") (at 99.06 41.275 90) (unit 1)
     (in_bom yes) (on_board yes) (dnp no) (fields_autoplaced)
     (property "Reference" "J2" (at 106.045 40.6399 90)
