File: zxmidi.kicad_pcb (KiCad board)
At the start: 2 copper layers, 53.1 x 21.7 mm, 6 parts, among them J1 RJ45, J2 DIN-5_180degree, Q1 BC337

Commit message: Case Upload
Parts:
- added REF**: MountingHole_2.5mm, MountingHole:MountingHole_2.5mm, F.Cu at (66.4, 53.9)
- added REF**: MountingHole_2.5mm, MountingHole:MountingHole_2.5mm, F.Cu at (66.4, 36.0)
Routing:
- net (no net): vias 2 -> 0
